Commit message: add 3dsensor support

File: ros_ws/src/pibot_description/urdf/hades.urdf (robot description, URDF)
Before this commit: robot pibot_description, 2 links, 1 joints
Links:
- added link 3dsensor_link, mass 0.17932; collision mesh filename=package://pibot_description/meshes/sensor/astra.dae; visual mesh filename=package://pibot_description/meshes/sensor/astra.dae
Joints:
- added joint 3dsensor_link_joint: type fixed, parent base_link, child 3dsensor_link, origin xyz=-0.1 0 0.125 rpy=1.2246E-16 -6.123E-17 0, axis 0 0 0

File: ros_ws/src/pibot_description/urdf/hera.urdf (robot description, URDF)
Before this commit: robot pibot_description, 2 links, 1 joints
Links:
- added link 3dsensor_link, mass 0.17932; collision mesh filename=package://pibot_description/meshes/sensor/astra.dae; visual mesh filename=package://pibot_description/meshes/sensor/astra.dae
Joints:
- added joint 3dsensor_link_joint: type fixed, parent base_link, child 3dsensor_link, origin xyz=-0.1 0 0.125 rpy=1.2246E-16 -6.123E-17 0, axis 0 0 0
