Commit message: update v1.1

File: ros_ws/src/pibot_description/urdf/apollo.urdf (robot description, URDF)
Before this commit: robot pibot_description, 2 links, 1 joints
Joints:
- joint laser_link_joint: origin xyz=-0.0525 0 0.09 rpy=0 0 0 -> xyz=0 0 0.09 rpy=0 0 0

File: ros_ws/src/pibot_description/urdf/zeus.urdf (robot description, URDF)
Before this commit: robot pibot_description, 2 links, 1 joints
Joints:
- joint laser_link_joint: type continuous -> fixed

Commit message: add 3d sensor model to apollo&zeus

File: ros_ws/src/pibot_description/urdf/apollo.urdf (robot description, URDF)
Before this commit: robot pibot_description, 2 links, 1 joints
Links:
- added link 3dsensor_link, mass 0.17932; collision mesh filename=package://pibot_description/meshes/sensor/astra.dae; visual mesh filename=package://pibot_description/meshes/sensor/astra.dae
Joints:
- added joint 3dsensor_link_joint: type fixed, parent base_link, child 3dsensor_link, origin xyz=-0.05 0 0.15 rpy=1.2246E-16 -6.123E-17 0, axis 0 0 0

File: ros_ws/src/pibot_description/urdf/apolloX.urdf (robot description, URDF)
Before this commit: robot pibot_description, 2 links, 1 joints
Links:
- added link 3dsensor_link, mass 0.17932; collision mesh filename=package://pibot_description/meshes/sensor/astra.dae; visual mesh filename=package://pibot_description/meshes/sensor/astra.dae
Joints:
- added joint 3dsensor_link_joint: type fixed, parent base_link, child 3dsensor_link, origin xyz=-0.05 0 0.25 rpy=1.2246E-16 -6.123E-17 0, axis 0 0 0

File: ros_ws/src/pibot_description/urdf/zeus.urdf (robot description, URDF)
Before this commit: robot pibot_description, 2 links, 1 joints
Links:
- added link 3dsensor_link, mass 0.17932; collision mesh filename=package://pibot_description/meshes/sensor/astra.dae; visual mesh filename=package://pibot_description/meshes/sensor/astra.dae
Joints:
- added joint 3dsensor_link_joint: type fixed, parent base_link, child 3dsensor_link, origin xyz=-0.1 0 0.25 rpy=1.2246E-16 -6.123E-17 0, axis 0 0 0

Commit message: depth camera

File: ros_ws/src/pibot_description/urdf/apollo.urdf (robot description, URDF)
Before this commit: robot pibot_description, 3 links, 2 joints
Links:
- removed link 3dsensor_link
- added link camera_link, mass 0.17932; collision mesh filename=package://pibot_description/meshes/sensor/astra.dae; visual mesh filename=package://pibot_description/meshes/sensor/astra.dae
Joints:
- removed joint 3dsensor_link_joint
- added joint camera_link_joint: type fixed, parent base_link, child camera_link, origin xyz=-0.05 0 0.15 rpy=1.2246E-16 -6.123E-17 0, axis 0 0 0

File: ros_ws/src/pibot_description/urdf/apolloX.urdf (robot description, URDF)
Before this commit: robot pibot_description, 3 links, 2 joints
Links:
- removed link 3dsensor_link
- added link camera_link, mass 0.17932; collision mesh filename=package://pibot_description/meshes/sensor/astra.dae; visual mesh filename=package://pibot_description/meshes/sensor/astra.dae
Joints:
- removed joint 3dsensor_link_joint
- added joint camera_link_joint: type fixed, parent base_link, child camera_link, origin xyz=-0.05 0 0.25 rpy=1.2246E-16 -6.123E-17 0, axis 0 0 0

File: ros_ws/src/pibot_description/urdf/hades.urdf (robot description, URDF)
Before this commit: robot pibot_description, 3 links, 2 joints
Links:
- removed link 3dsensor_link
- added link camera_link, mass 0.17932; collision mesh filename=package://pibot_description/meshes/sensor/astra.dae; visual mesh filename=package://pibot_description/meshes/sensor/astra.dae
Joints:
- removed joint 3dsensor_link_joint
- added joint camera_link_joint: type fixed, parent base_link, child camera_link, origin xyz=-0.1 0 0.125 rpy=1.2246E-16 -6.123E-17 0, axis 0 0 0

File: ros_ws/src/pibot_description/urdf/hera.urdf (robot description, URDF)
Before this commit: robot pibot_description, 3 links, 2 joints
Links:
- removed link 3dsensor_link
- added link camera_link, mass 0.17932; collision mesh filename=package://pibot_description/meshes/sensor/astra.dae; visual mesh filename=package://pibot_description/meshes/sensor/astra.dae
Joints:
- removed joint 3dsensor_link_joint
- added joint camera_link_joint: type fixed, parent base_link, child camera_link, origin xyz=-0.1 0 0.125 rpy=1.2246E-16 -6.123E-17 0, axis 0 0 0

File: ros_ws/src/pibot_description/urdf/zeus.urdf (robot description, URDF)
Before this commit: robot pibot_description, 3 links, 2 joints
Links:
- removed link 3dsensor_link
- added link camera_link, mass 0.17932; collision mesh filename=package://pibot_description/meshes/sensor/astra.dae; visual mesh filename=package://pibot_description/meshes/sensor/astra.dae
Joints:
- removed joint 3dsensor_link_joint
- added joint camera_link_joint: type fixed, parent base_link, child camera_link, origin xyz=-0.1 0 0.25 rpy=1.2246E-16 -6.123E-17 0, axis 0 0 0
